Commit message: Update mesh file path in hokuyo_ust10.urdf.xacro for correct referencing

File: urdf/hokuyo_ust10.urdf.xacro (robot description, xacro)
@@ -61,5 +61,5 @@
         <geometry>
           <!-- Origin of this mesh is the base of the bracket. -->
-          <mesh filename="package://urg_node/meshes/hokuyo_ust10.stl" />
+          <mesh filename="file://$(find urg_node)/meshes/hokuyo_ust10.stl"/>
         </geometry>
         <material name="dark_grey" />
